File: EAGLE/projects/Driver_TS_switch_latch/Driver_TS_switch_latch.brd (EAGLE design)
At the start: 24.1 x 39.4 mm, 3 parts, among them J1 T821108A1S100CEU, K1 EC2-12NU, K2 EC2-12NU

Commit message: Update for workshop
Signed-off-by: Jack Bruford <jack.bruford41@gmail.com>
Other:
- outline, holes or cut-outs redrawn
Changed lines of the file:
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@@
 <board>
 <plain>
-<wire x1="0" y1="0" x2="0" y2="38.1" width="0.127" layer="20"/>
-<wire x1="24.13" y1="38.1" x2="24.13" y2="0" width="0.127" layer="20"/>
+<wire x1="0" y1="0" x2="0" y2="39.37" width="0.127" layer="20"/>
+<wire x1="24.13" y1="39.37" x2="24.13" y2="0" width="0.127" layer="20"/>
 <wire x1="24.13" y1="0" x2="0" y2="0" width="0.127" layer="20"/>
-<wire x1="0" y1="38.1" x2="0" y2="39.37" width="0.127" layer="20"/>
 <wire x1="0" y1="39.37" x2="24.13" y2="39.37" width="0.127" layer="20"/>
-<wire x1="24.13" y1="39.37" x2="24.13" y2="38.1" width="0.127" layer="20"/>
 <text x="1.27" y="1.27" size="0.8128" layer="21">JACK BRUFORD - OXFORD UNI RACING
 DRIVER SWITCH INTERLOCK</text>
@@
 <wire x1="2.5972" y1="21.8723625" x2="3.81" y2="23.0851625" width="0.8128" layer="16"/>
 <wire x1="2.5972" y1="13.9128" x2="2.5972" y2="21.8723625" width="0.8128" layer="16"/>
-<wire x1="7.62" y1="8.89" x2="2.5972" y2="13.9128" width="0.8128" layer="16"/>
 <contactref element="J1" pad="3"/>
 <wire x1="7.62" y1="8.89" x2="10.16" y2="8.89" width="0.8128" layer="16"/>
+<wire x1="7.62" y1="8.89" x2="2.5972" y2="13.9128" width="0.8128" layer="16"/>
 </signal>
 <signal name="GND">
@@
 <wire x1="15.24" y1="24.35" x2="17.78" y2="24.35" width="0.8128" layer="16"/>
 <wire x1="17.78" y1="24.35" x2="20.32" y2="26.89" width="0.8128" layer="16"/>
-<wire x1="14.66680625" y1="7.5062" x2="15.81319375" y2="7.5062" width="0.8128" layer="16"/>
-<wire x1="15.81319375" y1="7.5062" x2="16.6238" y2="8.31680625" width="0.8128" layer="16"/>
-<wire x1="15.24" y1="13.38699375" x2="15.24" y2="24.35" width="0.8128" layer="16"/>
-<wire x1="16.6238" y1="8.31680625" x2="16.6238" y2="12.00319375" width="0.8128" layer="16"/>
-<wire x1="16.6238" y1="12.00319375" x2="15.24" y2="13.38699375" width="0.8128" layer="16"/>
-<wire x1="12.7" y1="8.89" x2="13.28300625" y2="8.89" width="0.8128" layer="16"/>
-<wire x1="13.28300625" y1="8.89" x2="14.66680625" y2="7.5062" width="0.8128" layer="16"/>
+<wire x1="14.6087375" y1="7.366" x2="15.8712625" y2="7.366" width="0.8128" layer="16"/>
+<wire x1="15.8712625" y1="7.366" x2="16.764" y2="8.2587375" width="0.8128" layer="16"/>
+<wire x1="16.764" y1="8.2587375" x2="16.764" y2="12.0612625" width="0.8128" layer="16"/>
+<wire x1="16.764" y1="12.0612625" x2="15.24" y2="13.5852625" width="0.8128" layer="16"/>
+<wire x1="12.7" y1="8.89" x2="13.0847375" y2="8.89" width="0.8128" layer="16"/>
+<wire x1="13.0847375" y1="8.89" x2="14.6087375" y2="7.366" width="0.8128" layer="16"/>
+<wire x1="15.24" y1="13.5852625" x2="15.24" y2="24.35" width="0.8128" layer="16"/>
 </signal>
 <signal name="ESDC-">
