File: EAGLE/projects/Oxford Uni Racing ECAD/Dashboard/Dashboard_Mid level design.sch (EAGLE design)
At the start: 0 parts

Commit message: updated buttons on all levels
Changed lines of the file:
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@@
 <port name="ASS1" side="top" coord="-22.86" direction="io"/>
 <port name="ASS2" side="top" coord="-20.32" direction="io"/>
-<port name="DISPL_SDA" side="top" coord="-15.24" direction="io"/>
-<port name="DISPL_SCL" side="top" coord="-12.7" direction="io"/>
 <port name="DRIVER_SELECT" side="top" coord="-7.62" direction="io"/>
 <port name="EVENT_SELECT" side="top" coord="-5.08" direction="io"/>
 <port name="PWR_REDUCTION" side="top" coord="0" direction="io"/>
 <port name="PEDAL_MAPPING" side="top" coord="2.54" direction="io"/>
-<port name="BRAKE_BIAS" side="top" coord="5.08" direction="io"/>
 <port name="TCS_ON_OFF" side="top" coord="10.16" direction="io"/>
 <port name="IGNITION_SWITCH" side="top" coord="15.24" direction="io"/>
-<port name="EMERGENCY_STOP" side="top" coord="20.32" direction="io"/>
+<port name="MISO" side="top" coord="20.32" direction="io"/>
+<port name="MOSI" side="top" coord="22.86" direction="io"/>
+<port name="DISPL_CS" side="top" coord="25.4" direction="io"/>
+<port name="SCK" side="top" coord="27.94" direction="io"/>
 </ports>
 <variantdefs>
@@
 <port name="CAN0" side="bottom" coord="-35.56" direction="io"/>
 <port name="CAN1" side="bottom" coord="-33.02" direction="io"/>
-<port name="DISPL_SDA" side="bottom" coord="-27.94" direction="io"/>
-<port name="DISPL_SCL" side="bottom" coord="-25.4" direction="io"/>
 <port name="DRIVER_SELECT" side="bottom" coord="-20.32" direction="io"/>
 <port name="EVENT_SELECT" side="bottom" coord="-17.78" direction="io"/>
 <port name="PWR_REDUCTION" side="bottom" coord="-12.7" direction="io"/>
 <port name="PEDAL_MAPPING" side="bottom" coord="-10.16" direction="io"/>
-<port name="BRAKE_BIAS" side="bottom" coord="-7.62" direction="io"/>
 <port name="TCS_ON_OFF" side="bottom" coord="-2.54" direction="io"/>
 <port name="IGNITION_SWITCH" side="bottom" coord="2.54" direction="io"/>
-<port name="EMERGENCY_STOP" side="bottom" coord="7.62" direction="io"/>
+<port name="MOSI" side="bottom" coord="12.7" direction="io"/>
+<port name="MISO" side="bottom" coord="15.24" direction="io"/>
+<port name="DISPL_CS" side="bottom" coord="17.78" direction="io"/>
+<port name="SCK" side="bottom" coord="20.32" direction="io"/>
 </ports>
 <variantdefs>
@@
 <port name="5V" side="bottom" coord="-12.7" direction="io"/>
 <port name="GND" side="bottom" coord="-10.16" direction="io"/>
-<port name="DISPL_SDA" side="bottom" coord="-5.08" direction="io"/>
-<port name="DISPL_SCL" side="bottom" coord="-2.54" direction="io"/>
+<port name="MOSI" side="bottom" coord="-5.08" direction="io"/>
+<port name="MISO" side="bottom" coord="-2.54" direction="io"/>
+<port name="CS" side="bottom" coord="0" direction="io"/>
+<port name="SCK" side="bottom" coord="2.54" direction="io"/>
 </ports>
 <variantdefs>
@@
 <port name="IGNITION_SWITCH" side="bottom" coord="-7.62" direction="io"/>
 <port name="PEDAL_MAPPING" side="bottom" coord="-2.54" direction="io"/>
-<port name="BRAKE_BIAS" side="bottom" coord="2.54" direction="io"/>
-<port name="EMERGENCY_STOP" side="bottom" coord="7.62" direction="io"/>
+<port name="TSMS" side="bottom" coord="2.54" direction="io"/>
 </ports>
 <variantdefs>
@@
 </instances>
 <busses>
-<bus name="3.3V,5V,12V,ASS1,ASS2,BRAKE_BIAS,CAN0,CAN1,DISPL_SCL,DISPL_SDA,DRIVER_SELECT,EMERGENCY_STOP,EVENT_SELECT,GND,IGNITION_SWITCH,PEDAL_MAPPING,PWR_REDUCTION,TCS_ON_OFF">
+<bus name="3.3V,5V,12V,ASS1,ASS2,CAN0,CAN1,DISPL_CS,DISPL_SCL,DRIVER_SELECT,EVENT_SELECT,GND,IGNITION_SWITCH,MISO,MOSI,PEDAL_MAPPING,PWR_REDUCTION,SCK,TCS_ON_OFF">
 <segment>
 <wire x1="332.74" y1="35.56" x2="327.66" y2="35.56" width="0.762" layer="92"/>
@@
 </segment>
 </net>
-<net name="DISPL_SDA" class="0">
-<segment>
-<portref moduleinst="MICROCONTROLLER1" port="DISPL_SDA"/>
-<wire x1="119.38" y1="35.56" x2="119.38" y2="45.72" width="0.1524" layer="91"/>
-</segment>
-<segment>
-<portref moduleinst="DISPLAY1" port="DISPL_SDA"/>
-<wire x1="213.36" y1="35.56" x2="213.36" y2="45.72" width="0.1524" layer="91"/>
-</segment>
-<segment>
-<portref moduleinst="INTER_SHEET_CONNECTIONS1" port="DISPL_SDA"/>
-<wire x1="96.52" y1="2.54" x2="96.52" y2="-5.08" width="0.1524" layer="91"/>
-</segment>
-</net>
 <net name="DISPL_SCL" class="0">
-<segment>
-<portref moduleinst="MICROCONTROLLER1" port="DISPL_SCL"/>
-<wire x1="121.92" y1="35.56" x2="121.92" y2="45.72" width="0.1524" layer="91"/>
-</segment>
 <segment>
 <portref moduleinst="DISPLAY1" port="GND"/>
 <wire x1="208.28" y1="35.56" x2="208.28" y2="45.72" width="0.1524" layer="91"/>
 </segment>
-<segment>
-<portref moduleinst="DISPLAY1" port="DISPL_SCL"/>
-<wire x1="215.9" y1="35.56" x2="215.9" y2="45.72" width="0.1524" layer="91"/>
-</segment>
-<segment>
-<portref moduleinst="INTER_SHEET_CONNECTIONS1" port="DISPL_SCL"/>
-<wire x1="99.06" y1="2.54" x2="99.06" y2="-5.08" width="0.1524" layer="91"/>
-</segment>
 </net>
 <net name="DRIVER_SELECT" class="0">
@@
 </segment>
 </net>
-<net name="BRAKE_BIAS" class="0">
-<segment>
-<portref moduleinst="MICROCONTROLLER1" port="BRAKE_BIAS"/>
-<wire x1="139.7" y1="35.56" x2="139.7" y2="45.72" width="0.1524" layer="91"/>
-</segment>
-<segment>
-<portref moduleinst="BUTTONS1" port="BRAKE_BIAS"/>
-<wire x1="284.48" y1="35.56" x2="284.48" y2="45.72" width="0.1524" layer="91"/>
-</segment>
-<segment>
-<portref moduleinst="INTER_SHEET_CONNECTIONS1" port="BRAKE_BIAS"/>
-<wire x1="116.84" y1="2.54" x2="116.84" y2="-5.08" width="0.1524" layer="91"/>
-</segment>
-</net>
 <net name="TCS_ON_OFF" class="0">
 <segment>
@@
 </segment>
 </net>
-<net name="EMERGENCY_STOP" class="0">
-<segment>
-<portref moduleinst="MICROCONTROLLER1" port="EMERGENCY_STOP"/>
-<wire x1="154.94" y1="35.56" x2="154.94" y2="45.72" width="0.1524" layer="91"/>
-</segment>
-<segment>
-<portref moduleinst="BUTTONS1" port="EMERGENCY_STOP"/>
-<wire x1="289.56" y1="35.56" x2="289.56" y2="45.72" width="0.1524" layer="91"/>
-</segment>
-<segment>
-<portref moduleinst="INTER_SHEET_CONNECTIONS1" port="EMERGENCY_STOP"/>
-<wire x1="132.08" y1="2.54" x2="132.08" y2="-5.08" width="0.1524" layer="91"/>
-</segment>
-</net>
 <net name="ASS1" class="0">
 <segment>
@@
 </segment>
 </net>
+<net name="MOSI" class="0">
+<segment>
+<portref moduleinst="MICROCONTROLLER1" port="MOSI"/>
+<wire x1="160.02" y1="45.72" x2="160.02" y2="35.56" width="0.1524" layer="91"/>
+</segment>
+<segment>
+<portref moduleinst="DISPLAY1" port="MOSI"/>
+<wire x1="213.36" y1="35.56" x2="213.36" y2="45.72" width="0.1524" layer="91"/>
+</segment>
+<segment>
+<portref moduleinst="INTER_SHEET_CONNECTIONS1" port="MOSI"/>
+<wire x1="134.62" y1="2.54" x2="134.62" y2="-5.08" width="0.1524" layer="91"/>
+</segment>
+</net>
+<net name="MISO" class="0">
+<segment>
+<portref moduleinst="MICROCONTROLLER1" port="MISO"/>
+<wire x1="162.56" y1="45.72" x2="162.56" y2="35.56" width="0.1524" layer="91"/>
+</segment>
+<segment>
+<portref moduleinst="DISPLAY1" port="MISO"/>
+<wire x1="215.9" y1="35.56" x2="215.9" y2="45.72" width="0.1524" layer="91"/>
+</segment>
+<segment>
+<portref moduleinst="INTER_SHEET_CONNECTIONS1" port="MISO"/>
+<wire x1="132.08" y1="2.54" x2="132.08" y2="-5.08" width="0.1524" layer="91"/>
+</segment>
+</net>
+<net name="DISPL_CS" class="0">
+<segment>
+<portref moduleinst="MICROCONTROLLER1" port="DISPL_CS"/>
+<wire x1="165.1" y1="45.72" x2="165.1" y2="35.56" width="0.1524" layer="91"/>
+</segment>
+<segment>
+<portref moduleinst="DISPLAY1" port="CS"/>
+<wire x1="218.44" y1="35.56" x2="218.44" y2="45.72" width="0.1524" layer="91"/>
+</segment>
+<segment>
+<portref moduleinst="INTER_SHEET_CONNECTIONS1" port="DISPL_CS"/>
+<wire x1="137.16" y1="2.54" x2="137.16" y2="-5.08" width="0.1524" layer="91"/>
+</segment>
+</net>
+<net name="SCK" class="0">
+<segment>
+<portref moduleinst="MICROCONTROLLER1" port="SCK"/>
+<wire x1="167.64" y1="45.72" x2="167.64" y2="35.56" width="0.1524" layer="91"/>
+</segment>
+<segment>
+<portref moduleinst="DISPLAY1" port="SCK"/>
+<wire x1="220.98" y1="35.56" x2="220.98" y2="45.72" width="0.1524" layer="91"/>
+</segment>
+<segment>
+<portref moduleinst="INTER_SHEET_CONNECTIONS1" port="SCK"/>
+<wire x1="139.7" y1="2.54" x2="139.7" y2="-5.08" width="0.1524" layer="91"/>
+</segment>
+</net>

Commit message: finilised ASS details
Changed lines of the file:
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@@
 <port name="DISPL_CS" side="top" coord="25.4" direction="io"/>
 <port name="SCK" side="top" coord="27.94" direction="io"/>
+<port name="TS" side="top" coord="33.02" direction="io"/>
 </ports>
 <variantdefs>
@@
 <port name="IGNITION_SWITCH" side="bottom" coord="-7.62" direction="io"/>
 <port name="PEDAL_MAPPING" side="bottom" coord="-2.54" direction="io"/>
-<port name="TSMS" side="bottom" coord="2.54" direction="io"/>
+<port name="TS" side="bottom" coord="2.54" direction="io"/>
 </ports>
 <variantdefs>
@@
 <port name="12V" side="bottom" coord="-12.7" direction="io"/>
 <port name="GND" side="bottom" coord="-10.16" direction="io"/>
+<port name="TS" side="bottom" coord="-7.62" direction="io"/>
+<port name="ASS1" side="bottom" coord="-2.54" direction="io"/>
+<port name="ASS2" side="bottom" coord="0" direction="io"/>
 </ports>
 <variantdefs>
@@
 </instances>
 <busses>
-<bus name="3.3V,5V,12V,ASS1,ASS2,CAN0,CAN1,DISPL_CS,DISPL_SCL,DRIVER_SELECT,EVENT_SELECT,GND,IGNITION_SWITCH,MISO,MOSI,PEDAL_MAPPING,PWR_REDUCTION,SCK,TCS_ON_OFF">
-<segment>
-<wire x1="332.74" y1="35.56" x2="327.66" y2="35.56" width="0.762" layer="92"/>
-<wire x1="327.66" y1="35.56" x2="58.42" y2="35.56" width="0.762" layer="92"/>
+<bus name="3.3V,5V,12V,ASS1,ASS2,CAN0,CAN1,DISPL_CS,DISPL_SCL,DRIVER_SELECT,EVENT_SELECT,GND,IGNITION_SWITCH,MISO,MOSI,PEDAL_MAPPING,PWR_REDUCTION,SCK,TCS_ON_OFF,TS">
+<segment>
+<wire x1="406.4" y1="35.56" x2="58.42" y2="35.56" width="0.762" layer="92"/>
 <wire x1="58.42" y1="35.56" x2="58.42" y2="2.54" width="0.762" layer="92"/>
 <wire x1="58.42" y1="2.54" x2="152.4" y2="2.54" width="0.762" layer="92"/>
-<wire x1="332.74" y1="35.56" x2="383.54" y2="35.56" width="0.762" layer="92"/>
 </segment>
 </bus>
@@
 <wire x1="58.42" y1="12.7" x2="48.26" y2="12.7" width="0.1524" layer="91"/>
 </segment>
+<segment>
+<portref moduleinst="TS_LATCH1" port="ASS1"/>
+<wire x1="388.62" y1="35.56" x2="388.62" y2="45.72" width="0.1524" layer="91"/>
+</segment>
 </net>
 <net name="ASS2" class="0">
@@
 <wire x1="58.42" y1="10.16" x2="48.26" y2="10.16" width="0.1524" layer="91"/>
 </segment>
+<segment>
+<portref moduleinst="TS_LATCH1" port="ASS2"/>
+<wire x1="391.16" y1="35.56" x2="391.16" y2="45.72" width="0.1524" layer="91"/>
+</segment>
 </net>
 <net name="MOSI" class="0">
@@
 </segment>
 </net>
+<net name="TS" class="0">
+<segment>
+<portref moduleinst="INTER_SHEET_CONNECTIONS1" port="TS"/>
+<wire x1="144.78" y1="-5.08" x2="144.78" y2="2.54" width="0.1524" layer="91"/>
+</segment>
+<segment>
+<portref moduleinst="BUTTONS1" port="TS"/>
+<wire x1="284.48" y1="45.72" x2="284.48" y2="35.56" width="0.1524" layer="91"/>
+</segment>
+<segment>
+<portref moduleinst="TS_LATCH1" port="TS"/>
+<wire x1="383.54" y1="35.56" x2="383.54" y2="45.72" width="0.1524" layer="91"/>
+</segment>
+</net>
