File: EAGLE/projects/Oxford Uni Racing ECAD/Wheel board/Wheel board.sch (EAGLE design)
At the start: 0 parts

Commit message: adding sheet to the low level desing for all modules, fixing top and mid level desing regarding motor controllers
Other:
- note added: "INTER_SHEET_CONNECTIONS"
