File: EAGLE/projects/Oxford Uni Racing ECAD/Top_Level_Design.sch (EAGLE design)
At the start: 0 parts

Commit message: updating mid and high level designs
Other:
- note added: "Double check telemetry"

Commit message: adding sheet to the low level desing for all modules, fixing top and mid level desing regarding motor controllers
Other:
- note removed: "Double check telemetry"
Changed lines of the file:
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@@
 <port name="ASS2" side="bottom" coord="15.24" direction="io"/>
 <port name="CURRENT_SENSE_PLAUSABILITY" side="bottom" coord="22.86" direction="io"/>
+<port name="STEERING_WHEEL_POSITION_S" side="top" coord="0" direction="io"/>
 </ports>
 <variantdefs>
@@
 <port name="ASS1" side="top" coord="5.08" direction="io"/>
 <port name="ASS2" side="top" coord="7.62" direction="io"/>
-<port name="TELEM_1" side="right" coord="7.62" direction="io"/>
-<port name="TELEM_2" side="right" coord="5.08" direction="io"/>
 <port name="MOTOR_CONTR_L_1" side="left" coord="5.08" direction="io"/>
-<port name="MOTOR_CONTR_L_2" side="left" coord="2.54" direction="io"/>
 <port name="MOTOR_CONTR_R_1" side="left" coord="-5.08" direction="io"/>
-<port name="MOTOR_CONTR_R_2" side="left" coord="-7.62" direction="io"/>
-<port name="PWR_OUT" side="right" coord="2.54" direction="io"/>
-<port name="GND_OUT" side="right" coord="0" direction="io"/>
 </ports>
 <variantdefs>
@@
 <module name="MOTOR_CONTROLLER" prefix="" dx="30.48" dy="20.32">
 <ports>
-<port name="LINE_1" side="right" coord="-2.54" direction="io"/>
-<port name="LINE_2" side="right" coord="-5.08" direction="io"/>
+<port name="DATA" side="right" coord="-2.54" direction="io"/>
 </ports>
 <variantdefs>
@@
 </sheets>
 </module>
+<module name="STEERING_WHEEL_POSITION" prefix="" dx="30.48" dy="20.32">
+<ports>
+<port name="PWR" side="right" coord="-7.62" direction="io"/>
+<port name="GND" side="right" coord="-5.08" direction="io"/>
+<port name="OUT" side="right" coord="5.08" direction="io"/>
+</ports>
+<variantdefs>
+</variantdefs>
+<parts>
+</parts>
+<sheets>
+<sheet>
+<plain>
+</plain>
+<instances>
+</instances>
+<busses>
+</busses>
+<nets>
+</nets>
+</sheet>
+</sheets>
+</module>
 </modules>
 <parts>
@@
 <sheet>
 <plain>
-<text x="162.56" y="-55.88" size="1.778" layer="91">Double check telemetry</text>
 </plain>
 <moduleinsts>
@@
 <attribute name="NAME" x="165.1" y="195.58" size="2.032" layer="95" align="bottom-center"/>
 </moduleinst>
-<moduleinst name="TELEMETRY1" module="TELEMETRY" x="175.26" y="-40.64">
-<attribute name="NAME" x="175.26" y="-40.64" size="2.032" layer="95" align="bottom-center"/>
-</moduleinst>
 <moduleinst name="MOTOR_CONTROLLER1" module="MOTOR_CONTROLLER" x="2.54" y="-35.56">
 <attribute name="NAME" x="2.54" y="-35.56" size="2.032" layer="95" align="bottom-center"/>
@@
 <attribute name="NAME" value="LV_MASTER_SWITCH" x="342.9" y="-7.62" size="2.032" layer="95" rot="R180" align="bottom-center"/>
 </moduleinst>
+<moduleinst name="STEERING_WHEEL_POSITION1" module="STEERING_WHEEL_POSITION" x="165.1" y="170.18">
+<attribute name="NAME" x="165.1" y="170.18" size="2.032" layer="95" align="bottom-center"/>
+</moduleinst>
 </moduleinsts>
 <instances>
@@
 <wire x1="-66.04" y1="10.16" x2="213.36" y2="10.16" width="0.762" layer="92"/>
 <label x="86.36" y="7.62" size="1.778" layer="95"/>
+</segment>
+</bus>
+<bus name="B$1">
+<segment>
+<wire x1="55.88" y1="-40.64" x2="40.64" y2="-40.64" width="0.762" layer="92"/>
+<wire x1="40.64" y1="-40.64" x2="40.64" y2="-38.1" width="0.762" layer="92"/>
+<wire x1="40.64" y1="-38.1" x2="22.86" y2="-38.1" width="0.762" layer="92"/>
+</segment>
+</bus>
+<bus name="B$2">
+<segment>
+<wire x1="22.86" y1="-63.5" x2="40.64" y2="-63.5" width="0.762" layer="92"/>
+<wire x1="40.64" y1="-63.5" x2="40.64" y2="-50.8" width="0.762" layer="92"/>
+<wire x1="40.64" y1="-50.8" x2="55.88" y2="-50.8" width="0.762" layer="92"/>
 </segment>
 </bus>
@@
 <wire x1="185.42" y1="111.76" x2="193.04" y2="111.76" width="0.1524" layer="91"/>
 <junction x="193.04" y="111.76"/>
+<portref moduleinst="STEERING_WHEEL_POSITION1" port="PWR"/>
+<wire x1="193.04" y1="137.16" x2="193.04" y2="162.56" width="0.1524" layer="91"/>
+<wire x1="193.04" y1="162.56" x2="185.42" y2="162.56" width="0.1524" layer="91"/>
+<junction x="193.04" y="137.16"/>
 </segment>
 </net>
@@
 <wire x1="185.42" y1="114.3" x2="195.58" y2="114.3" width="0.1524" layer="91"/>
 <junction x="195.58" y="114.3"/>
+<portref moduleinst="STEERING_WHEEL_POSITION1" port="GND"/>
+<wire x1="185.42" y1="165.1" x2="195.58" y2="165.1" width="0.1524" layer="91"/>
+<wire x1="195.58" y1="165.1" x2="195.58" y2="139.7" width="0.1524" layer="91"/>
+<junction x="195.58" y="139.7"/>
 </segment>
 </net>
@@
 <portref moduleinst="THROTTLE_PEDAL_2" port="PWR"/>
 <wire x1="289.56" y1="45.72" x2="314.96" y2="45.72" width="0.1524" layer="91"/>
-</segment>
-</net>
-<net name="N$30" class="0">
-<segment>
-<portref moduleinst="VCU1" port="PWR_OUT"/>
-<portref moduleinst="TELEMETRY1" port="PWR"/>
-<wire x1="116.84" y1="-43.18" x2="154.94" y2="-43.18" width="0.1524" layer="91"/>
-</segment>
-</net>
-<net name="N$31" class="0">
-<segment>
-<portref moduleinst="TELEMETRY1" port="GND"/>
-<portref moduleinst="VCU1" port="GND_OUT"/>
-<wire x1="154.94" y1="-45.72" x2="116.84" y2="-45.72" width="0.1524" layer="91"/>
-</segment>
-</net>
-<net name="N$32" class="0">
-<segment>
-<portref moduleinst="VCU1" port="TELEM_2"/>
-<wire x1="116.84" y1="-40.64" x2="144.78" y2="-40.64" width="0.1524" layer="91"/>
-<wire x1="144.78" y1="-40.64" x2="144.78" y2="-38.1" width="0.1524" layer="91"/>
-<portref moduleinst="TELEMETRY1" port="DATA_?"/>
-<wire x1="144.78" y1="-38.1" x2="154.94" y2="-38.1" width="0.1524" layer="91"/>
-</segment>
-</net>
-<net name="N$33" class="0">
-<segment>
-<portref moduleinst="VCU1" port="TELEM_1"/>
-<wire x1="116.84" y1="-38.1" x2="142.24" y2="-38.1" width="0.1524" layer="91"/>
-<wire x1="142.24" y1="-38.1" x2="142.24" y2="-35.56" width="0.1524" layer="91"/>
-<portref moduleinst="TELEMETRY1" port="CLOCK_?"/>
-<wire x1="142.24" y1="-35.56" x2="154.94" y2="-35.56" width="0.1524" layer="91"/>
-</segment>
-</net>
-<net name="N$34" class="0">
-<segment>
-<portref moduleinst="VCU1" port="MOTOR_CONTR_L_1"/>
-<wire x1="55.88" y1="-40.64" x2="43.18" y2="-40.64" width="0.1524" layer="91"/>
-<wire x1="43.18" y1="-40.64" x2="43.18" y2="-38.1" width="0.1524" layer="91"/>
-<portref moduleinst="MOTOR_CONTROLLER1" port="LINE_1"/>
-<wire x1="43.18" y1="-38.1" x2="22.86" y2="-38.1" width="0.1524" layer="91"/>
-</segment>
-</net>
-<net name="N$35" class="0">
-<segment>
-<portref moduleinst="VCU1" port="MOTOR_CONTR_L_2"/>
-<wire x1="55.88" y1="-43.18" x2="40.64" y2="-43.18" width="0.1524" layer="91"/>
-<wire x1="40.64" y1="-43.18" x2="40.64" y2="-40.64" width="0.1524" layer="91"/>
-<portref moduleinst="MOTOR_CONTROLLER1" port="LINE_2"/>
-<wire x1="40.64" y1="-40.64" x2="22.86" y2="-40.64" width="0.1524" layer="91"/>
-</segment>
-</net>
-<net name="N$36" class="0">
-<segment>
-<portref moduleinst="VCU1" port="MOTOR_CONTR_R_2"/>
-<wire x1="55.88" y1="-53.34" x2="43.18" y2="-53.34" width="0.1524" layer="91"/>
-<wire x1="43.18" y1="-53.34" x2="43.18" y2="-66.04" width="0.1524" layer="91"/>
-<portref moduleinst="MOTOR_CONTROLLER2" port="LINE_2"/>
-<wire x1="43.18" y1="-66.04" x2="22.86" y2="-66.04" width="0.1524" layer="91"/>
-</segment>
-</net>
-<net name="N$37" class="0">
-<segment>
-<portref moduleinst="MOTOR_CONTROLLER2" port="LINE_1"/>
-<wire x1="22.86" y1="-63.5" x2="40.64" y2="-63.5" width="0.1524" layer="91"/>
-<wire x1="40.64" y1="-63.5" x2="40.64" y2="-50.8" width="0.1524" layer="91"/>
-<portref moduleinst="VCU1" port="MOTOR_CONTR_R_1"/>
-<wire x1="40.64" y1="-50.8" x2="55.88" y2="-50.8" width="0.1524" layer="91"/>
 </segment>
 </net>
@@
 </segment>
 </net>
+<net name="N$30" class="0">
+<segment>
+<portref moduleinst="STEERING_WHEEL_POSITION1" port="OUT"/>
+<portref moduleinst="PEDAL_BOARD1" port="STEERING_WHEEL_POSITION_S"/>
+<wire x1="185.42" y1="175.26" x2="220.98" y2="175.26" width="0.1524" layer="91"/>
+<wire x1="220.98" y1="175.26" x2="220.98" y2="71.12" width="0.1524" layer="91"/>
+</segment>
+</net>
