File: EAGLE/projects/Oxford Uni Racing ECAD/Pedal board/Pedal board_Mid level design.sch (EAGLE design)
At the start: 0 parts

Commit message: adding sheet to the low level desing for all modules, fixing top and mid level desing regarding motor controllers
Changed lines of the file:
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@@
 <port name="ASS2" side="top" coord="2.54" direction="io"/>
 <port name="BATT_CURR" side="top" coord="7.62" direction="io"/>
+<port name="ST_WH_POSS" side="top" coord="12.7" direction="io"/>
 </ports>
 <variantdefs>
@@
 <port name="BR_POSS" side="bottom" coord="0" direction="io"/>
 <port name="BRAKE_LIGHTS_OUT" side="bottom" coord="5.08" direction="io"/>
+<port name="ST_WHEEL_POSS" side="bottom" coord="10.16" direction="io"/>
 </ports>
 <variantdefs>
@@
 </sheets>
 </module>
+<module name="STEERING_WHEEL_POSS" prefix="" dx="30.48" dy="20.32">
+<ports>
+<port name="3.3V" side="bottom" coord="-12.7" direction="io"/>
+<port name="GND" side="bottom" coord="-10.16" direction="io"/>
+<port name="ST_WH_POSS" side="bottom" coord="0" direction="io"/>
+</ports>
+<variantdefs>
+</variantdefs>
+<parts>
+</parts>
+<sheets>
+<sheet>
+<plain>
+</plain>
+<instances>
+</instances>
+<busses>
+</busses>
+<nets>
+</nets>
+</sheet>
+</sheets>
+</module>
 </modules>
 <parts>
@@
 <attribute name="NAME" x="353.06" y="50.8" size="2.032" layer="95" align="bottom-center"/>
 </moduleinst>
+<moduleinst name="STEERING_WHEEL_POSS1" module="STEERING_WHEEL_POSS" x="398.78" y="50.8">
+<attribute name="NAME" x="398.78" y="50.8" size="2.032" layer="95" align="bottom-center"/>
+</moduleinst>
 </moduleinsts>
 <instances>
 </instances>
 <busses>
-<bus name="3.3V,5V,12V,ASS1,ASS2,BATT_CURR_SENSE,BRAKE_LIGHTS_OUT,BR_POSS,BR_PR,CAN0,CAN1,GND,THR1,THR2,THR3">
-<segment>
-<wire x1="43.18" y1="22.86" x2="353.06" y2="22.86" width="0.762" layer="92"/>
+<bus name="3.3V,5V,12V,ASS1,ASS2,BATT_CURR_SENSE,BRAKE_LIGHTS_OUT,BR_POSS,BR_PR,CAN0,CAN1,GND,ST_WH_POSS,THR1,THR2,THR3">
+<segment>
+<wire x1="43.18" y1="22.86" x2="414.02" y2="22.86" width="0.762" layer="92"/>
 <wire x1="43.18" y1="22.86" x2="43.18" y2="-12.7" width="0.762" layer="92"/>
 <wire x1="43.18" y1="-12.7" x2="165.1" y2="-12.7" width="0.762" layer="92"/>
@@
 <wire x1="342.9" y1="22.86" x2="342.9" y2="35.56" width="0.1524" layer="91"/>
 </segment>
+<segment>
+<portref moduleinst="STEERING_WHEEL_POSS1" port="GND"/>
+<wire x1="388.62" y1="22.86" x2="388.62" y2="35.56" width="0.1524" layer="91"/>
+</segment>
 </net>
 <net name="CAN0" class="0">
@@
 <wire x1="83.82" y1="-12.7" x2="83.82" y2="-22.86" width="0.1524" layer="91"/>
 </segment>
+<segment>
+<portref moduleinst="STEERING_WHEEL_POSS1" port="3.3V"/>
+<wire x1="386.08" y1="22.86" x2="386.08" y2="35.56" width="0.1524" layer="91"/>
+</segment>
 </net>
 <net name="THR1" class="0">
@@
 </segment>
 </net>
+<net name="ST_WH_POSS" class="0">
+<segment>
+<portref moduleinst="STEERING_WHEEL_POSS1" port="ST_WH_POSS"/>
+<wire x1="398.78" y1="35.56" x2="398.78" y2="22.86" width="0.1524" layer="91"/>
+</segment>
+<segment>
+<portref moduleinst="MICROCONTROLLER1" port="ST_WHEEL_POSS"/>
+<wire x1="114.3" y1="22.86" x2="114.3" y2="35.56" width="0.1524" layer="91"/>
+</segment>
+<segment>
+<portref moduleinst="CROSS_SHEET_WIRING1" port="ST_WH_POSS"/>
+<wire x1="134.62" y1="-12.7" x2="134.62" y2="-22.86" width="0.1524" layer="91"/>
+</segment>
+</net>
