File: EAGLE/projects/Oxford Uni Racing ECAD/Pedal board/Pedal board_Mid level design.sch (EAGLE design)
At the start: 0 parts

Commit message: removed throttle position sensor 3 from all chematics
Changed lines of the file:
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@@
 <port name="THR1" side="top" coord="-22.86" direction="io"/>
 <port name="THR2" side="top" coord="-20.32" direction="io"/>
-<port name="THR3" side="top" coord="-17.78" direction="io"/>
 <port name="BR_PR" side="top" coord="-12.7" direction="io"/>
 <port name="BR_POSS" side="top" coord="-10.16" direction="io"/>
@@
 <port name="THR1" side="bottom" coord="-12.7" direction="io"/>
 <port name="THR2" side="bottom" coord="-10.16" direction="io"/>
-<port name="THR3" side="bottom" coord="-7.62" direction="io"/>
 <port name="BR_PR" side="bottom" coord="-2.54" direction="io"/>
 <port name="BR_POSS" side="bottom" coord="0" direction="io"/>
@@
 <port name="THR_POSS1" side="bottom" coord="-5.08" direction="io"/>
 <port name="THR_POSS2" side="bottom" coord="-2.54" direction="io"/>
-<port name="THR_POSS3" side="bottom" coord="0" direction="io"/>
 <port name="BR_POSS" side="bottom" coord="2.54" direction="io"/>
 <port name="BR_PRESS" side="bottom" coord="5.08" direction="io"/>
@@
 </segment>
 </net>
-<net name="THR3" class="0">
-<segment>
-<portref moduleinst="MICROCONTROLLER1" port="THR3"/>
-<wire x1="96.52" y1="22.86" x2="96.52" y2="35.56" width="0.1524" layer="91"/>
-</segment>
-<segment>
-<portref moduleinst="CROSS_SHEET_WIRING1" port="THR3"/>
-<wire x1="104.14" y1="-12.7" x2="104.14" y2="-22.86" width="0.1524" layer="91"/>
-</segment>
-<segment>
-<portref moduleinst="OUTPUTS1" port="THR_POSS3"/>
-<wire x1="154.94" y1="22.86" x2="154.94" y2="35.56" width="0.1524" layer="91"/>
-</segment>
-</net>
