File: EAGLE/projects/Oxford Uni Racing ECAD/Control Panel/Control Panel.brd (EAGLE design)
At the start: 160 x 100 mm, 37 parts

Commit message: Created Control Panel Board and edited holes lbr so that the name apears on the silkscreen layer
Signed-off-by: Jack Bruford <jack.bruford@oxforduniracing.com>
Parts:
- moved LVB+_MP 453.5 mm to (-130.8, 151.1)
- moved GLV+_MP 437.9 mm to (-100.3, 151.1)
- moved ASS- 437.2 mm to (-53.3, 176.5)
- moved GLV-_MP 436.9 mm to (-66.0, 163.8)
- moved ASS+ 426.1 mm to (-30.5, 176.5)
- moved R1 411.5 mm to (-67.3, 171.4)
- moved LED1 406.5 mm to (-82.5, 172.7)
- moved HV_CONTROL_UNIT_SUPPLY 403.9 mm to (-72.4, 74.9)
- moved HV_CONTROL_UNIT_GND 398.8 mm to (-66.0, 87.6)
- moved COOLING_PUMP_GND 338.0 mm to (-59.7, 113.0)
- moved F8 322.7 mm to (-80.0, 8.89)
- moved INS_GND 309.2 mm to (-36.8, 163.8)
- moved LV_BATTERY_SUPPLY 307.6 mm to (-59.7, 125.7)
- moved COOLING_PUMP_SUPPLY 304.7 mm to (-125.7, 87.6)
- moved LV_MASTER_SWITCH+ 273.3 mm to (-118.1, 100.3)
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