File: EAGLE/projects/Oxford Uni Racing ECAD/HV Battery/power electronics2.sch (EAGLE design)
At the start: 28 parts, among them IC1 4043N, IC2 4001N, K1 T9AS1D12-48=T9A, K2 T9AS5D12-12=T9A, K4 T9AS1D12-48=T9A, K5 T9AS1D12-48=T9A

Commit message: Commiting power electronics files Signed-off-by: Jack Bruford <jack.bruford@oxforduniracing.com>
Parts:
- added C1, C2: (no value), rcl:C-EU050-024X044
- added IC3: LM555CN, SamacSys_Parts:LM555CN
- added IC4: 4071N, 40xx:4071N
- added Q1, Q2: BSS92, transistor-fet:BSS92
- added R4: 10K, rcl:R-EU_0207/15
Connections:
- new net IMD_LED_OUT: MISC_I/O.3, Q1.D
- new net N$18: C2.1, IC3.DISCHARGE, IC3.THRESHOLD, R4.1
- new net N$19: C1.1, IC3.CONTROL_VOLTAGE
- new net N$20: IC1A.R0, IC3.OUTPUT
- new net N$21: IC1A.Q0, IC4A.I1, Q2.G
- new net N$22: IC4A.O, Q1.G
- net +12V: now also IC1P.VDD, IC2P.VDD, IC3.RESET, IC3.TRIGGER, IC3.VCC, IC4P.VDD, Q1.S, Q2.S, R4.2
- net GND: now also C1.2, C2.2, IC1P.VSS, IC2P.VSS, IC3.GND, IC4P.VSS, MISC_I/O.4; no longer IC1A.R0
- net N$11: now also IC4A.I0
- net N$15: now also Q2.D; no longer IC1A.Q0
Other:
- moved on the sheet: D5, HV+, HV_INDICATOR, R1
