File: EAGLE/projects/Oxford Uni Racing ECAD/HV Battery/power electronics3.brd (EAGLE design)
At the start: 191.8 x 114 mm, 57 parts, among them IC1 4043N, IC2 4001N, IC3 LM555CN, IC4 4071N, IC5 4081N, IC6 4011N, IC7 4011N, K1 T9AS1D12-48=T9A, K2 T9AS5D12-12=T9A, K4 T9AS1D12-48=T9A, K5 T9AS1D12-48=T9A, Q1 BS170, Q2 BS170, Q3 BS170

Commit message: Modifications suggested by Dan after first review
Signed-off-by: Jack Bruford <jack.bruford41@gmail.com>
Parts:
- removed S1: MOMENTARY-SWITCH-SPST-PTH-6.0MM, SparkFun-Switches:TACTILE_SWITCH_PTH_6.0MM
- Q2: value BS170 -> BSS92; device transistor-small-signal:SOT54E -> transistor-fet:TO92
- moved Q3 84.1 mm to (135.9, 78.7)
- moved Q1 82.5 mm to (69.8, 29.2)
- moved Q2 38.7 mm to (68.6, 19.1), turned to 270 degrees
- moved TP10 27.9 mm to (154.9, 69.8)
- moved EMSDC 15.2 mm to (14.0, 14.0)
- moved EMSDC_POSAIR- 2.54 mm to (14.0, 67.3)
Connections:
- removed net N$36: IC5.1, IC7.8, TP10.TP
- removed net N$37: IC6.11, Q2.G
- new net VDD: IC5.14, IC6.14, IC7.14
- new net VSS: IC5.7, IC6.7, IC7.7
- net +12V: now also Q2.3; no longer IC5.7, IC6.7, IC7.7, Q2.S, S1.1
- net CHG_SAFE: now also IC5.1, IC6.12, IC6.13, TP10.TP; no longer IC7.9
- net EMSDC_IMD+: now also K1.4; no longer K1.3
- net GND: no longer IC5.14, IC6.14, IC7.14
- net N$15: now also Q2.2; no longer Q2.D
- net N$16: now also K1.3; no longer K1.4
- net N$20: no longer S1.3
- net N$21: now also Q2.1; no longer IC6.12, IC6.13
- net N$32: now also IC6.11; no longer IC7.10
Routing:
- net VDD: track 0.00 -> 84.8 mm
- net VSS: track 0.00 -> 43.6 mm
- net CHG_SAFE: track 232.3 -> 265.5 mm
- net N$15: track 22.8 -> 39.9 mm
- net N$16: track 8.89 -> 25.9 mm
- net EMSDC_IMD+: track 59.7 -> 71.1 mm
- net N$21: track 106.5 -> 117.3 mm
- net +12V: track 395.2 -> 404.7 mm
- net N$36: track 8.67 -> 0.00 mm
- net N$2: track 158.0 -> 154.0 mm
- net N$23: track 153.9 -> 155.2 mm
- net N$32: track 49.7 -> 50.8 mm
- net GND: track 340.7 -> 341.5 mm
