File: EAGLE/projects/Oxford Uni Racing ECAD/HV Battery/power electronics4.brd (EAGLE design)
At the start: 191.8 x 114 mm, 57 parts, among them IC1 4043N, IC2 4001N, IC3 LM555CN, IC4 4071N, IC5 4081N, IC6 4011N, IC7 4011N, K1 T9AS1D12-48=T9A, K2 T9AS5D12-12=T9A, K4 T9AS1D12-48=T9A, K5 T9AS1D12-48=T9A, Q1 BS170, Q2 BS170, Q3 BS170

Commit message: Modifications suggested by Dan after first review
Signed-off-by: Jack Bruford <jack.bruford41@gmail.com>
Parts:
- removed IC2: 4001N, 40xx:DIL14
- removed IC4: 4071N, 40xx:DIL14
- removed IC5: 4081N, 40xx:DIL14
- removed IC7: 4011N, 40xx:DIL14
- removed S1: MOMENTARY-SWITCH-SPST-PTH-6.0MM, SparkFun-Switches:TACTILE_SWITCH_PTH_6.0MM
- removed TP10, TP5, TP9: TPSPAD1-17, testpad:P1-17
- added C3: 50uF, rcl:C050-024X044
- added R5: 10K, rcl:0207/15
- added R6: 50K, rcl:0207/15
- added R7: 500K, rcl:0207/15
- C1: value (none) -> 0.1uF
- C2: value (none) -> 220uF
Connections:
- removed net N$23: IC1.6, IC5.4, TP7.TP
- removed net N$24: IC6.3, IC6.5, IC6.6
- removed net N$25: IC6.4, IC6.8, IC6.9
- removed net N$26: IC5.6, IC6.10
- removed net N$27: IC1.12, IC5.3, TP8.TP
- removed net N$28: IC5.2, IC7.4
- removed net N$29: IC1.10, IC4.6
- removed net N$30: IC7.3, IC7.5, IC7.6
- removed net N$32: IC7.1, IC7.10, IC7.2
- removed net N$34: IC4.4, Q1.G
- removed net N$36: IC5.1, IC7.8, TP10.TP
- new net VDD: IC6.14
- new net VSS: IC6.7
- net +12V: now also R6.2; no longer IC2.14, IC3.2, IC4.14, IC5.7, IC6.7, IC7.7, S1.1
- net CHG_SAFE: now also IC1.12, TP8.TP; no longer IC7.9
- net DISCHARGE_ENABLE: now also IC1.6, TP7.TP; no longer IC5.5, IC6.1, IC6.2, TP9.TP
- net GND: now also C3.2, R5.1, R7.1; no longer IC2.7, IC4.7, IC5.14, IC6.14, IC7.14
- net N$11: now also IC1.11, IC1.3, IC1.7, IC3.3, R5.2, TP4.TP; no longer IC2.1, IC2.12, IC2.13, IC4.1, ISOMETER_INPUTS.8, R2.1, TP5.TP
- net N$12: now also IC1.9, IC6.5, IC6.6, TP3.TP; no longer IC2.11, IC2.8, IC2.9
- net N$13: now also IC1.10, IC6.8, IC6.9; no longer IC2.10, IC2.5, IC2.6
- net N$14: now also IC6.1, IC6.4; no longer IC2.2, IC2.4
- net N$17: now also ISOMETER_INPUTS.8, R2.1; no longer IC2.3
- net N$20: now also IC6.10, IC6.2; no longer IC1.11, IC1.3, IC1.7, IC3.3, S1.3, TP4.TP
- net N$21: now also IC6.3, Q1.G; no longer IC1.2, IC4.2, IC6.12, IC6.13, TP2.TP
- net N$22: now also C3.1, IC3.2, R6.1, R7.2; no longer IC1.9, IC4.5, TP3.TP
- net N$35: now also IC1.2, IC6.12, IC6.13, TP2.TP; no longer IC4.3
Routing:
- net N$23: track 153.9 -> 0.00 mm
- net DISCHARGE_ENABLE: track 157.6 -> 275.1 mm
- net N$11: track 144.7 -> 28.3 mm, vias 2 -> 0
- net N$35: track 0.00 -> 106.5 mm, vias 0 -> 2
- net N$21: track 106.5 -> 0.00 mm, vias 2 -> 0
- net N$32: track 49.7 -> 0.00 mm
- net +12V: track 395.2 -> 345.7 mm
- net N$27: track 44.9 -> 0.00 mm
- net CHG_SAFE: track 232.3 -> 276.0 mm
- net N$28: track 37.4 -> 0.00 mm
- net N$20: track 36.0 -> 0.00 mm
- net GND: track 340.7 -> 316.6 mm
- net N$12: track 13.8 -> 0.00 mm
- net N$24: track 13.8 -> 0.00 mm
- net N$25: track 13.0 -> 0.00 mm
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