File: EAGLE/projects/Oxford Uni Racing ECAD/HV Battery/power electronics6.sch (EAGLE design)
At the start: 57 parts, among them IC1 4043N, IC2 4001N, IC3 LM555CN, IC4 4071N, IC5 4081N, IC6 4011N, IC7 4011N, K1 T9AS1D12-48=T9A, K2 T9AS5D12-12=T9A, K4 T9AS1D12-48=T9A, K5 T9AS1D12-48=T9A, Q1 BS170, Q2 BS170, Q3 BS170

Commit message: Modifications suggested by Dan after first review
Signed-off-by: Jack Bruford <jack.bruford41@gmail.com>
Parts:
- removed BMS_INPUTS, ISOMETER_INPUTS: T821108A1S100CEU, SamacSys_Parts:T821108A1S100CEU
- removed C1, C2: (no value), rcl:C-EU050-024X044
- removed D3, D4: 1N4004, diode:1N4004
- removed EMSDC_POSAIR-, EMSDC_PRECHARGERELAY-, EMSDC_TSMS+, EMSDC_TSMS-, GND, GND1, HV+, HV_INDICATOR: MOUNT-PAD-ROUND3.0, holes:MOUNT-PAD-ROUND3.0
- removed IC3: LM555CN, SamacSys_Parts:LM555CN
- removed IC5: 4081N, 40xx:4081N
- removed IC7: 4011N, 40xx:4011N
- removed S1: MOMENTARY-SWITCH-SPST-PTH-6.0MM, SparkFun-Switches:MOMENTARY-SWITCH-SPST-PTH-6.0MM
- removed TP10, TP4, TP5, TP9: TPSPAD1-17, testpad:TPSPAD1-17
- removed X1: (no value), con-wago-508:W237-3E
- added AIR_AUX, POWER/GND: (no value), con-molex:KK-156-3
- added BMS_I/O, ISOMETER_I/O, THERAL_EX_I/O, WIFI_I/O: T821108A1S100CEU, SamacSys_Parts:T821108A1S100CEU
- added C4: 3.3uF, rcl:C-EUC1206
- added C5: 1uF, rcl:C-EUC1206
- added C6: 0.1uF, rcl:C-EUC1206
- added C7: 220uF, rcl:C-EUC1206
- added C8: 50uF, rcl:C-EUC1206
- added D2: VS-30BQ100-M3_9AT, SamacSys_Parts:VS-30BQ100-M3_9AT
- added FAN-, J12: 8191, SamacSys_Parts:8191
- added K3: T9AS1D12-48=T9A, SamacSys_Parts:T9AS1D12-48=T9A
- added PRECHARGE/AIRS: (no value), con-molex:KK-156-6
- added R10: 50K, rcl:R-EU_R1206
- added R11: 500K, rcl:R-EU_R1206
- added R5, R9: 10K, rcl:R-EU_R1206
- added R6, R7: 2.2K, rcl:R-EU_R1206
- D1, D6, D7, D8: value 1N4004 -> ES2D; device diode:1N4004 -> diode:ES2D
- D5: value 1N5369BRLG -> VS-30BQ100-M3_9AT; device SamacSys_Parts:1N5369BRLG -> SamacSys_Parts:VS-30BQ100-M3_9AT
- EMSDC: value MOUNT-PAD-ROUND3.0 -> (none); device holes:MOUNT-PAD-ROUND3.0 -> con-molex:KK-156-6
- IC1: value 4043N -> 4043D; device 40xx:4043N -> 40xx:4043D
- IC2: value 4001N -> SE555D; device 40xx:4001N -> linear:SE555D
- IC4: value 4071N -> (none); device 40xx:4071N -> linear-technology:LT1129CS8
- IC6: value 4011N -> 4011D; device 40xx:4011N -> 40xx:4011D
- R1: value 3.3K -> 120; device rcl:R-EU_0207/15 -> rcl:R-EU_R1206
- R2, R3: device rcl:R-EU_0207/12 -> rcl:R-EU_R1206
- R4: value 10K -> 120; device rcl:R-EU_0207/15 -> rcl:R-EU_R1206
Connections:
- net AMS_LED_OUT renamed AMS_LED-
- net IMD_LED_OUT renamed IMD_LED-
- removed net N$16: EMSDC.MOUNT, K1.NO
- removed net N$18: C2.1, IC3.DISCHARGE, IC3.THRESHOLD, R4.1
- removed net N$22: IC1A.Q1, IC4B.I0, TP3.PP
- removed net N$23: IC1A.S1, IC5B.O, TP7.PP
- removed net N$24: IC6A.O, IC6B.I0, IC6B.I1
- removed net N$25: IC6B.O, IC6C.I0, IC6C.I1
- removed net N$26: IC5B.I1, IC6C.O
- removed net N$27: IC1A.S2, IC5A.O, TP8.PP
- removed net N$29: IC1A.Q2, IC4B.I1
- removed net N$30: IC7A.O, IC7B.I0, IC7B.I1
- removed net N$31: F2.2, X1-2.KL
- removed net N$33: F1.2, X1-1.KL
- removed net N$34: IC4B.O, Q1.G
- removed net N$35: IC4A.O, Q3.G
- removed net N$36: IC5A.I0, IC7C.I0, TP10.PP
- removed net N$5: D5.K, HV+.MOUNT
- removed net N$6: BMS_INPUTS.3, D3.A, F2.1
- removed net N$7: D5.A, R1.2
- removed net N$9: HV_INDICATOR.MOUNT, R1.1
- removed net PRECHARGE/SS_SELECT: BMS_INPUTS.1, D1.C, K2.4
- new net +3V3: C4.1, IC1A.EN, IC1P.VDD, IC2.R, IC2.V+, IC4G$1.OUT, IC4G$1.SENSE, IC6P.VDD, R10.2, R5.2, R6.1, R7.1
- new net AMS_COIL_OUT: D8.A, K1.COIL_2, Q2.D
- new net CAN2_H: BMS_I/O.6, MISC_I/O.7, R1.1, R4.1, THERAL_EX_I/O.3, WIFI_I/O.3
- new net CAN2_L: BMS_I/O.8, MISC_I/O.8, R1.2, R4.2, THERAL_EX_I/O.5, WIFI_I/O.5
- new net CHARGE_POWER: BMS_I/O.3, D5.A, F1.1, THERAL_EX_I/O.2, WIFI_I/O.2
- new net CHARGE_SAFE: D6.A, K5.COIL_1
- new net CHASSIS_GND: ISOMETER_I/O.3, MISC_I/O.1
- new net DISCHARE_ENABLE: IC1A.S1, R7.2, TP7.PP
- new net FAN+: J12.1, J12.2, J12.3, J12.4, K3.NO
- new net FAN_ENABLE: BMS_I/O.5, K3.COIL_2
- new net HIGHEST_TEMP: THERAL_EX_I/O.4
- new net LOWEST_TEMP: THERAL_EX_I/O.6
- new net M_HS: ISOMETER_I/O.5, R3.1, TP1.PP
- new net OK_HS: IC1A.S0, ISOMETER_I/O.8, R2.1, TP6.PP
- new net PRECHARGE_SELECT: BMS_I/O.7, D1.C, K2.4
- new net READY_POWER: BMS_I/O.1, D2.A, F2.1, THERAL_EX_I/O.1, WIFI_I/O.1
- new net STARTUP_RESET: IC1A.R0, IC1A.R1, IC1A.R2, IC2.Q, R9.2
- net +12V: now also AIR_AUX-1.S, AIR_AUX-2.S, AIR_AUX-3.S, C5.1, D2.K, D5.K, D8.C, IC4G$1.IN, ISOMETER_I/O.2, K1.COIL_1, K3.COIL_1, K3.COM, K4.COIL_1, K5.COIL_2, MISC_I/O.2, MISC_I/O.4; no longer D3.C, D4.C, GND1.MOUNT, IC1A.EN, IC1P.VDD, IC2P.VDD, IC3.RESET, IC3.TRIGGER, IC3.VCC, IC4P.VDD, IC5P.VSS, IC6P.VSS, IC7P.VSS, ISOMETER_INPUTS.2, K4.COIL_2, K5.COIL_1, MISC_I/O.1, Q1.S, Q2.S, Q3.S, R4.2, S1.1
- net CHG_SAFE: now also BMS_I/O.2, IC1A.S2, R6.2, TP8.PP; no longer BMS_INPUTS.2, D6.A, IC7C.I1, K5.COIL_2
- net DISCHARGE_ENABLE: now also BMS_I/O.4, K4.COIL_2; no longer BMS_INPUTS.4, IC5B.I0, IC6A.I0, IC6A.I1, K4.COIL_1, TP9.PP
- net GND: now also C4.2, C5.2, C6.2, C7.2, C8.2, FAN-.1, FAN-.2, FAN-.3, FAN-.4, IC1A.R3, IC1A.S3, IC2.GND, IC4G$1.GND, IC6P.VSS, ISOMETER_I/O.1, POWER/GND-3.S, PRECHARGE/AIRS-3.S, PRECHARGE/AIRS-4.S, PRECHARGE/AIRS-6.S, Q1.S, Q2.S, Q3.S, R11.1, R9.1, THERAL_EX_I/O.8, WIFI_I/O.8; no longer C1.2, C2.2, D8.A, GND.MOUNT, IC2P.VSS, IC3.GND, IC4P.VSS, IC5P.VDD, IC6P.VDD, IC7P.VDD, ISOMETER_INPUTS.1, K1.COIL_2, MISC_I/O.4, MISC_I/O.8, X1-3.KL
- net N$1: now also EMSDC-1.S, K4.COM, K5.NO; no longer EMSDC_TSMS-.MOUNT, K2.1
- net N$10: now also IC1A.Q1, IC6B.I0, IC6B.I1, TP3.PP; no longer ISOMETER_INPUTS.5, R3.1, TP1.PP
- net N$11: now also EMSDC-5.S, K2.1, PRECHARGE/AIRS-5.S; no longer IC2A.I0, IC2D.I0, IC2D.I1, IC4A.I0, ISOMETER_INPUTS.8, R2.1, TP5.PP
- net N$12: now also K2.3, PRECHARGE/AIRS-2.S; no longer IC2C.I0, IC2C.I1, IC2D.O
- net N$13: now also IC1A.Q2, IC6C.I0, IC6C.I1; no longer IC2B.I0, IC2B.I1, IC2C.O
- net N$14: now also IC6A.I0, IC6B.O; no longer IC2A.I1, IC2B.O
- net N$15: now also EMSDC-2.S, K1.NO; no longer D8.C, K1.COIL_1, Q2.D
- net N$17: now also C7.1, IC2.DIS, IC2.THR, R5.1; no longer IC1A.S0, IC2A.O, TP6.PP
- net N$19: now also EMSDC-3.S, EMSDC-4.S; no longer C1.1, IC3.CONTROL_VOLTAGE
- net N$2: now also F2.2, POWER/GND-2.S; no longer EMSDC_POSAIR-.MOUNT, K2.3
- net N$20: now also IC6A.I1, IC6C.O; no longer IC1A.R0, IC1A.R1, IC1A.R2, IC3.OUTPUT, S1.2, TP4.PP
- net N$21: now also IC6A.O, Q1.G; no longer IC1A.Q0, IC4A.I1, IC6D.I0, IC6D.I1, TP2.PP
- net N$28: now also C8.1, IC2.TR, R10.1, R11.2; no longer IC5A.I1, IC7B.O
- net N$3: now also PRECHARGE/AIRS-1.S; no longer EMSDC_PRECHARGERELAY-.MOUNT
- net N$32: now also C6.1, IC2.CV; no longer IC7A.I0, IC7A.I1, IC7C.O
- net N$4: now also F1.2, POWER/GND-1.S; no longer EMSDC_TSMS+.MOUNT, K4.COM, K5.NO
- net N$8: now also IC1A.Q0, IC6D.I0, IC6D.I1, Q3.G, TP2.PP; no longer BMS_INPUTS.5, D4.A, F1.1
Other:
- note added: "1: Chassis GND (LV connector) 2: IMD LED + (LV connector) 3: IMD LED - (LV connector) 4: AMS LED + (LV connector) 5: AMS LED - (LV connector) 6: NC 7: CAN2 H (LV connector) 8: CAN2 L (LV connector)"
- note added: "1: EMSDC (LV connector) 2: EMSDC MSD/HVIL+ (Lid Mounted) 3: EMSDC MSD/HVIL- (Lid Mounted) 4: EMSDC TSMS+(LV connector) 5: EMSDC TSMS-(LV connector) 6: NC"
- note added: "1: GND (for supply) 2: 12V Supply 3: Chassis GND 4: NC 5: M_HS (PWM status signal) 6: NC 7: NC 8: OK_HS (logic signal)"
- note added: "1: Positive AIR+ 2: Precharge Relay + 3: Positive AIR- 4: Precharge Relay- 5: Negative AIR+ 6: Negative AIR-"
- note added: "1: Ready Power (LV connector) 2: Charge Power (LV connector) 3: GND (LV connector)"
- note added: "1: Ready Power 2: Charge Power 3: CAN2 H 4: Higest Temp (NC) 5: CAN2_L 6: Lowest Temp (NC) 7: NC 8: GND"
- note added: "1: Ready Power 2: Charge Power 3: CAN2 H 4: NC 5: CAN2 L 6: NC 7: NC 8: GND"
- note added: "1: Ready Power BMS input 2: Charge Safe BMS Output 3: Charge Power BMS input 4: Discharge_Enable BMS Output 5: Fan_Enable 6: CAN 2 H 7: Prechage select (Multi-Purpose Enbale) 8: CAN 2 L"
- note added: "Combined Power Supply: 5 x T821 relays: 83mA*5=0.42A Fan: 2A Isometer: 150mA AMS LED: 20mA BMS LED: 20mA Total: 2.6A Selected diode rated to 3A"
- note added: "Maximum permissable fuse: 5A"
- note added: "Monostable Reset Pulse (this pulse must exceeed the startup time of the BMS and IMD, the length of the pulse should be considered the startup time for the board). Pulse duration: 2.5s"
- note added: "Need to use opto couples for 12V signals if regulating it at 3.3v"
- note added: "No termination resistor built in for CAN2 in either BMS or Thermal Expansion Module, require two 120 ohm resistors on network MAY NOT BE REQUIRED IF INSTALLED ON OTHER DEVICES ON NETWORK"
- note added: "Switch Mode regulator input bypass capacitor used as reccomended for circuits powered from a battery voltage source in the application notes"
- note removed: "Monostable Reset Pulse Generator"
- note removed: "Negative edge detection"
- note removed: "positive edge detection"
- moved on the sheet: F1, F2, H1, H2, H3, H4, IC1, IC1P, IC6A, IC6B, IC6C, IC6D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
