File: EAGLE/projects/Oxford Uni Racing ECAD/HV Battery/power electronics6.brd (EAGLE design)
At the start: 191.8 x 114 mm, 57 parts, among them IC1 4043N, IC2 4001N, IC3 LM555CN, IC4 4071N, IC5 4081N, IC6 4011N, IC7 4011N, K1 T9AS1D12-48=T9A, K2 T9AS5D12-12=T9A, K4 T9AS1D12-48=T9A, K5 T9AS1D12-48=T9A, Q1 BS170, Q2 BS170, Q3 BS170

Commit message: Modifications suggested by Dan after first review
Signed-off-by: Jack Bruford <jack.bruford41@gmail.com>
Parts:
- removed C1, C2: (no value), rcl:C050-024X044
- removed D3, D4: 1N4004, diode:DO41-10
- removed EMSDC_POSAIR-, EMSDC_PRECHARGERELAY-, EMSDC_TSMS+, EMSDC_TSMS-, GND, GND1, HV+, HV_INDICATOR: MOUNT-PAD-ROUND3.0, holes:3,0-PAD
- removed IC3: LM555CN, SamacSys_Parts:DIP762W53P254L980H533Q8N
- removed IC5: 4081N, 40xx:DIL14
- removed IC7: 4011N, 40xx:DIL14
- removed ISOMETER_INPUTS: T821108A1S100CEU, SamacSys_Parts:HDRV8W64P254_2X4_1778X895X915P
- removed S1: MOMENTARY-SWITCH-SPST-PTH-6.0MM, SparkFun-Switches:TACTILE_SWITCH_PTH_6.0MM
- removed TP10, TP4, TP5, TP9: TPSPAD1-17, testpad:P1-17
- removed X1: (no value), con-wago-508:W237-3E
- added AIR_AUX, POWER/GND: (no value), con-molex:KK-156-3
- added C4: 3.3uF, rcl:C1206
- added C5: 1uF, rcl:C1206
- added C6: 0.1uF, rcl:C1206
- added C7: 220uF, rcl:C1206
- added C8: 50uF, rcl:C1206
- added D2: VS-30BQ100-M3_9AT, SamacSys_Parts:DIOM7959X262N
- added FAN-, J12: 8191, SamacSys_Parts:8191
- added ISOMETER_I/O, THERAL_EX_I/O, WIFI_I/O: T821108A1S100CEU, SamacSys_Parts:HDRV8W64P254_2X4_1778X895X915P
- added K3: T9AS1D12-48=T9A, SamacSys_Parts:T9AS1D1248T9A
- added PRECHARGE/AIRS: (no value), con-molex:KK-156-6
- added R10: 50K, rcl:R1206
- added R11: 500K, rcl:R1206
- added R5, R9: 10K, rcl:R1206
- added R6, R7: 2.2K, rcl:R1206
- D1, D6, D7, D8: value 1N4004 -> ES2D; device diode:DO41-10 -> diode:SMB
- D5: value 1N5369BRLG -> VS-30BQ100-M3_9AT; device SamacSys_Parts:DIOAD2260W109L864D349 -> SamacSys_Parts:DIOM7959X262N
- EMSDC: value MOUNT-PAD-ROUND3.0 -> (none); device holes:3,0-PAD -> con-molex:KK-156-6
- IC1: value 4043N -> 4043D; device 40xx:DIL16 -> 40xx:SO16
- IC2: value 4001N -> SE555D; device 40xx:DIL14 -> linear:SO08
- IC4: value 4071N -> (none); device 40xx:DIL14 -> linear-technology:SOIC8
- IC6: value 4011N -> 4011D; device 40xx:DIL14 -> 40xx:SO14
- R1: value 3.3K -> 120; device rcl:0207/15 -> rcl:R1206
- R2, R3: device rcl:0207/12 -> rcl:R1206
- R4: value 10K -> 120; device rcl:0207/15 -> rcl:R1206
- moved R1 455.5 mm to (-223.5, -130.8), turned to 0 degrees
- moved D5 451.1 mm to (-224.8, -152.4), turned to 0 degrees
- moved R4 364.4 mm to (-223.5, -137.2), turned to 0 degrees
- moved EMSDC 301.5 mm to (-219.7, -161.3)
- moved IC4 180.8 mm to (-15.2, -27.9)
- moved IC2 172.9 mm to (-41.9, -45.7)
- renumbered BMS_INPUTS to BMS_I/O
Connections:
- net AMS_LED_OUT renamed AMS_LED-
- net IMD_LED_OUT renamed IMD_LED-
- removed net N$16: EMSDC.B3,0, K1.4
- removed net N$18: C2.1, IC3.6, IC3.7, R4.1
- removed net N$22: IC1.9, IC4.5, TP3.TP
- removed net N$23: IC1.6, IC5.4, TP7.TP
- removed net N$24: IC6.3, IC6.5, IC6.6
- removed net N$25: IC6.4, IC6.8, IC6.9
- removed net N$26: IC5.6, IC6.10
- removed net N$27: IC1.12, IC5.3, TP8.TP
- removed net N$29: IC1.10, IC4.6
- removed net N$30: IC7.3, IC7.5, IC7.6
- removed net N$31: F2.2, X1.2
- removed net N$33: F1.2, X1.1
- removed net N$34: IC4.4, Q1.G
- removed net N$35: IC4.3, Q3.G
- removed net N$36: IC5.1, IC7.8, TP10.TP
- removed net N$5: D5.1, HV+.B3,0
- removed net N$6: BMS_I/O.3, D3.A, F2.1
- removed net N$7: D5.2, R1.2
- removed net N$9: HV_INDICATOR.B3,0, R1.1
- removed net PRECHARGE/SS_SELECT: BMS_I/O.1, D1.C, K2.4
- new net +3V3: C4.1, IC1.16, IC1.5, IC2.4, IC2.8, IC4.1, IC4.2, IC6.14, R10.2, R5.2, R6.1, R7.1
- new net AMS_COIL_OUT: D8.A, K1.2, Q2.D
- new net CAN2_H: BMS_I/O.6, MISC_I/O.7, R1.1, R4.1, THERAL_EX_I/O.3, WIFI_I/O.3
- new net CAN2_L: BMS_I/O.8, MISC_I/O.8, R1.2, R4.2, THERAL_EX_I/O.5, WIFI_I/O.5
- new net CHARGE_POWER: BMS_I/O.3, D5.2, F1.1, THERAL_EX_I/O.2, WIFI_I/O.2
- new net CHARGE_SAFE: D6.A, K5.1
- new net CHASSIS_GND: ISOMETER_I/O.3, MISC_I/O.1
- new net DISCHARE_ENABLE: IC1.6, R7.2, TP7.TP
- new net FAN+: J12.1, J12.2, J12.3, J12.4, K3.4
- new net FAN_ENABLE: BMS_I/O.5, K3.2
- new net HIGHEST_TEMP: THERAL_EX_I/O.4
- new net LOWEST_TEMP: THERAL_EX_I/O.6
- new net M_HS: ISOMETER_I/O.5, R3.1, TP1.TP
- new net OK_HS: IC1.4, ISOMETER_I/O.8, R2.1, TP6.TP
- new net PRECHARGE_SELECT: BMS_I/O.7, D1.C, K2.4
- new net READY_POWER: BMS_I/O.1, D2.2, F2.1, THERAL_EX_I/O.1, WIFI_I/O.1
- new net STARTUP_RESET: IC1.11, IC1.3, IC1.7, IC2.3, R9.2
- net +12V: now also AIR_AUX.1, AIR_AUX.2, AIR_AUX.3, C5.1, D2.1, D5.1, D8.C, IC4.8, ISOMETER_I/O.2, K1.1, K3.1, K3.3, K4.1, K5.2, MISC_I/O.2, MISC_I/O.4; no longer D3.C, D4.C, GND1.B3,0, IC1.16, IC1.5, IC2.14, IC3.2, IC3.4, IC3.8, IC4.14, IC5.7, IC6.7, IC7.7, ISOMETER_INPUTS.2, K4.2, K5.1, MISC_I/O.1, Q1.S, Q2.S, Q3.S, R4.2, S1.1
- net CHG_SAFE: now also IC1.12, R6.2, TP8.TP; no longer D6.A, IC7.9, K5.2
- net DISCHARGE_ENABLE: now also K4.2; no longer IC5.5, IC6.1, IC6.2, K4.1, TP9.TP
- net GND: now also C4.2, C5.2, C6.2, C7.2, C8.2, FAN-.1, FAN-.2, FAN-.3, FAN-.4, IC1.14, IC1.15, IC2.1, IC4.3, IC4.6, IC6.7, ISOMETER_I/O.1, POWER/GND.3, PRECHARGE/AIRS.3, PRECHARGE/AIRS.4, PRECHARGE/AIRS.6, Q1.S, Q2.S, Q3.S, R11.1, R9.1, THERAL_EX_I/O.8, WIFI_I/O.8; no longer C1.2, C2.2, D8.A, GND.B3,0, IC2.7, IC3.1, IC5.14, IC6.14, IC7.14, ISOMETER_INPUTS.1, K1.2, MISC_I/O.4, MISC_I/O.8, X1.3
- net N$1: now also EMSDC.1, K4.3, K5.4; no longer EMSDC_TSMS-.B3,0, K2.1
- net N$10: now also IC1.9, IC6.5, IC6.6, TP3.TP; no longer ISOMETER_INPUTS.5, R3.1, TP1.TP
- net N$11: now also EMSDC.5, K2.1, PRECHARGE/AIRS.5; no longer IC2.1, IC2.12, IC2.13, IC4.1, ISOMETER_INPUTS.8, R2.1, TP5.TP
- net N$12: now also K2.3, PRECHARGE/AIRS.2; no longer IC2.11, IC2.8, IC2.9
- net N$13: now also IC1.10, IC6.8, IC6.9; no longer IC2.10, IC2.5, IC2.6
- net N$14: now also IC6.1, IC6.4; no longer IC2.2, IC2.4
- net N$15: now also EMSDC.2, K1.4; no longer D8.C, K1.1, Q2.D
- net N$17: now also C7.1, IC2.6, IC2.7, R5.1; no longer IC1.4, IC2.3, TP6.TP
- net N$19: now also EMSDC.3, EMSDC.4; no longer C1.1, IC3.5
- net N$2: now also F2.2, POWER/GND.2; no longer EMSDC_POSAIR-.B3,0, K2.3
- net N$20: now also IC6.10, IC6.2; no longer IC1.11, IC1.3, IC1.7, IC3.3, S1.3, TP4.TP
- net N$21: now also IC6.3, Q1.G; no longer IC1.2, IC4.2, IC6.12, IC6.13, TP2.TP
- net N$28: now also C8.1, IC2.2, R10.1, R11.2; no longer IC5.2, IC7.4
- net N$3: now also PRECHARGE/AIRS.1; no longer EMSDC_PRECHARGERELAY-.B3,0
- net N$32: now also C6.1, IC2.5; no longer IC7.1, IC7.10, IC7.2
- net N$4: now also F1.2, POWER/GND.1; no longer EMSDC_TSMS+.B3,0, K4.3, K5.4
- net N$8: now also IC1.2, IC6.12, IC6.13, Q3.G, TP2.TP; no longer BMS_I/O.5, D4.A, F1.1
Routing:
- net +12V: track 395.2 -> 0.00 mm, vias 1 -> 0
- net GND: track 340.7 -> 111.6 mm
- net CHG_SAFE: track 232.3 -> 44.4 mm
- net PRECHARGE_SELECT: track 0.00 -> 169.2 mm
- net PRECHARGE/SS_SELECT: track 168.0 -> 0.00 mm
- net N$2: track 158.0 -> 0.00 mm
- net DISCHARGE_ENABLE: track 157.6 -> 0.00 mm
- net DISCHARE_ENABLE: track 0.00 -> 154.9 mm
- net N$23: track 153.9 -> 0.00 mm
- net N$11: track 144.7 -> 0.00 mm, vias 2 -> 0
- net N$12: track 13.8 -> 155.5 mm
- net N$21: track 106.5 -> 0.00 mm, vias 2 -> 0
- net N$6: track 81.8 -> 0.00 mm
- net N$1: track 109.6 -> 28.9 mm
- net M_HS: track 0.00 -> 61.1 mm
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
Commit message: Updated to include discharge/dischare enable bug, amended 555 passive compoenent values to match values in deptartment stores
Signed-off-by: Jack Bruford <jack.bruford41@gmail.com>
Parts:
- removed FAN-, J12: 8191, SamacSys_Parts:8191
- removed TP1, TP2, TP3, TP6, TP7, TP8: TPSPAD1-17, testpad:P1-17
- added D3: ES2D, diode:SMB
- added FAN: (no value), con-molex:KK-156-2
- Q1, Q2, Q3: value BS170 -> BSS138; device transistor-small-signal:SOT54E -> m-pad-2.1:SOT23
- moved THERAL_EX_I/O 441.9 mm to (170.2, 104.1)
- moved WIFI_I/O 430.6 mm to (148.6, 104.1)
- moved AIR_AUX 416.7 mm to (66.0, 105.4), turned to 180 degrees
- moved R6 406.6 mm to (116.8, 7.62)
- moved R7 406.6 mm to (116.8, 1.27)
- moved PRECHARGE/AIRS 382.7 mm to (40.6, 105.4)
- moved K3 356.8 mm to (154.9, 35.6)
- moved R4 339.5 mm to (14.0, 105.4), turned to 180 degrees
- moved R1 330.5 mm to (14.0, 99.1), turned to 180 degrees
- moved D5 326.6 mm to (50.8, 22.9)
- moved D2 325.5 mm to (50.8, 34.3)
- moved EMSDC 320.7 mm to (14.0, 58.4), turned to 90 degrees
- moved POWER/GND 320.2 mm to (14.0, 31.8), turned to 90 degrees
- moved C8 200.8 mm to (130.8, 14.0), turned to 270 degrees
- moved R11 197.6 mm to (123.2, 14.0), turned to 90 degrees
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Connections:
- net +12V: now also D3.C
- net AMS_COIL_OUT: now also Q2.3; no longer Q2.D
- net AMS_LED-: now also Q1.3; no longer Q1.D
- net CHG_SAFE: no longer TP8.TP
- net DISCHARE_ENABLE: no longer TP7.TP
- net FAN+: now also FAN.1; no longer J12.1, J12.2, J12.3, J12.4
- net FAN_ENABLE: now also D3.A
- net GND: now also FAN.2, Q1.2, Q2.2, Q3.2; no longer FAN-.1, FAN-.2, FAN-.3, FAN-.4, Q1.S, Q2.S, Q3.S
- net IMD_LED-: now also Q3.3; no longer Q3.D
- net M_HS: no longer TP1.TP
- net N$10: no longer TP3.TP
- net N$21: now also Q1.1; no longer Q1.G
- net N$37: now also Q2.1; no longer Q2.G
- net N$8: now also Q3.1; no longer Q3.G, TP2.TP
- net OK_HS: no longer TP6.TP
Routing:
- net N$12: track 155.5 -> 0.00 mm
- net DISCHARE_ENABLE: track 154.9 -> 0.00 mm
- net +12V: track 0.00 -> 119.4 mm
- net N$3: track 93.6 -> 0.00 mm
- net PRECHARGE_SELECT: track 169.2 -> 79.6 mm
- net GND: track 111.6 -> 33.2 mm
- net AMS_LED-: track 71.9 -> 0.00 mm
- net M_HS: track 61.1 -> 0.00 mm
- net EMSDC_IMD+: track 59.7 -> 0.00 mm
- net IMD_LED-: track 54.4 -> 0.00 mm
- net CAN2_L: track 0.00 -> 50.0 mm
- net CAN2_H: track 0.00 -> 46.6 mm
- net CHG_SAFE: track 44.4 -> 0.00 mm
- net OK_HS: track 37.5 -> 0.00 mm
- net N$1: track 28.9 -> 0.00 mm
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- removed copper zone on layer 1, net GND
- removed copper zone on layer 16, net GND
