File: EAGLE/projects/Oxford Uni Racing ECAD/HV Battery/AccumulatorMainBoard/power electronicsV4.3.brd (EAGLE design)
At the start: 167.6 x 103.8 mm, 94 parts, among them IC1 4043D, IC2 SE555D, IC9 4011D, K2 T9AS5D12-12=T9A, K3 T9AS1D12-48=T9A, K6 T9AS1D12-48=T9A, K7 T9AS1D12-48=T9A, Q1 BSS138, Q2 BSS138, Q3 BSS138, Q4 BSS138

Commit message: Mainboard .brd file updates
Routed all the wires to the connector. and solves DRC conflicts.
Parts:
- moved THERMAL_EX_I/0 461.3 mm to (124.5, 99.1)
- moved BMS_I/O 444.7 mm to (8.89, 86.4), turned to 90 degrees
- moved PRECHARGE 322.1 mm to (7.62, 20.3), turned to 137.5 degrees
- moved ISOMETER_I/O 305.9 mm to (128.3, 5.08), turned to 180 degrees
- moved MISC_I/O 257.3 mm to (10.2, 40.6), turned to 270 degrees
- moved WIFI_MODULE 178.3 mm to (19.1, 99.1), turned to 180 degrees
- moved K7 150.9 mm to (67.3, 61.0), turned to 180 degrees
- moved TP9 108.9 mm to (134.6, 100.3)
- moved TP8 107.6 mm to (133.3, 101.6)
- moved K6 94.8 mm to (35.6, 58.4), turned to 180 degrees
Connections:
- removed net AMS_LED: MISC_I/O.5
- removed net IMD_LED: MISC_I/O.3
- net AMS_LED-: now also MISC_I/O.5
- net IMD_LED-: now also MISC_I/O.3
Routing:
- net CAN2_H: track 9.62 -> 293.8 mm, vias 0 -> 2
- net CAN2_L: track 10.9 -> 288.0 mm, vias 0 -> 2
- net CAN1_L: track 75.2 -> 216.7 mm, vias 0 -> 1
- net PRECHARGE_SELECT: track 43.9 -> 182.7 mm
- net CAN1_H: track 81.8 -> 220.4 mm, vias 0 -> 2
- net CHASSIS_GND: track 0.00 -> 138.6 mm
- net PRECHARGE_EMSDC2: track 0.00 -> 124.6 mm, vias 0 -> 3
- net N$21: track 0.00 -> 59.9 mm
- net READY_POWER: track 216.5 -> 270.6 mm, vias 3 -> 5
- net PRECHARGE_EMSDC1: track 0.00 -> 52.4 mm, vias 0 -> 1
- net CHARGE_POWER: track 208.6 -> 252.4 mm, vias 3 -> 4
- net DISCHARGE_ENABLE: track 112.8 -> 146.5 mm
- net OK_HS: track 131.4 -> 162.6 mm
- net LOWEST_TEMP: track 0.00 -> 22.4 mm
- net FAN_ENABLE: track 95.2 -> 115.3 mm
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