File: EAGLE/projects/Oxford Uni Racing ECAD/HV Battery/AccumulatorMainBoard/power electronicsV5.1.brd (EAGLE design)
At the start: 167.6 x 103.8 mm, 84 parts, among them IC1 4043D, IC2 SE555D, IC9 4011D, K2 T9AS5D12-12=T9A, K6 T9AS1D12-48=T9A, K7 T9AS1D12-48=T9A, Q1 BSS138, Q2 BSS138, Q3 BSS138, Q4 BSS138

Commit message: final fnl... mainbaord
yeah
Parts:
- renumbered LED4-DISCHARGE-ENABLE to LED4, LED5-CHARGE-SAFE to LED5
Other:
- board text added: "Charge-Safe"
- board text added: "Designed by: Xianming Liu, James Willy, Aminah Dixon, Omar Ahmed Accumulator Mainboard V2"
- board text added: "Discharge-enable"
- board text removed: "Designed by: Xianming Liu, James Willy, Aminah Dixon, Omar Ahmed"
